File: Voice Modulator/voicemodulator_schm.sch (EAGLE design)
At the start: 26 parts, among them T1 2N5089, T2 2N5089, T3 2N5089, T4 2N5089

Commit message: Add ISP pin to schematic
Parts:
- added ISP: (no value), con-lstb:MA03-2
Connections:
- new net N$22: ATMEGA48AIC.PC6(!RESET!/PCINT14), ISP.2
- net 0: now also ISP.1
- net N$16: now also ISP.3
- net N$17: now also ISP.4
- net N$2: now also ISP.6
- net VCC: now also ISP.5
Changed lines of the file:
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@@
 <part name="P+4" library="audio amplifier example" library_urn="urn:adsk.eagle:library:970892" deviceset="VCC" device=""/>
 <part name="P+5" library="audio amplifier example" library_urn="urn:adsk.eagle:library:970892" deviceset="VCC" device=""/>
+<part name="ISP" library="con-lstb" library_urn="urn:adsk.eagle:library:162" deviceset="MA03-2" device="" package3d_urn="urn:adsk.eagle:package:8334/1"/>
+<part name="X_10" library="ngspice-simulation" library_urn="urn:adsk.eagle:library:527439" deviceset="GND" device=""/>
+<part name="P+6" library="audio amplifier example" library_urn="urn:adsk.eagle:library:970892" deviceset="VCC" device=""/>
 </parts>
 <sheets>
@@
 </instance>
 <instance part="X_1" gate="G$1" x="165.1" y="63.5" smashed="yes"/>
-<instance part="X_2" gate="G$1" x="45.72" y="2.54" smashed="yes"/>
-<instance part="P+1" gate="VCC" x="88.9" y="22.86" smashed="yes">
-<attribute name="VALUE" x="87.376" y="23.876" size="1.27" layer="96"/>
+<instance part="X_2" gate="G$1" x="50.8" y="2.54" smashed="yes"/>
+<instance part="P+1" gate="VCC" x="86.36" y="22.86" smashed="yes">
+<attribute name="VALUE" x="84.836" y="23.876" size="1.27" layer="96"/>
 </instance>
 <instance part="R1" gate="G$1" x="132.08" y="60.96" smashed="yes" rot="R90">
@@
 <instance part="P+5" gate="VCC" x="-35.56" y="35.56" smashed="yes">
 <attribute name="VALUE" x="-37.084" y="36.576" size="1.27" layer="96"/>
+</instance>
+<instance part="ISP" gate="1" x="38.1" y="-22.86" smashed="yes">
+<attribute name="VALUE" x="34.29" y="-30.48" size="1.778" layer="96"/>
+<attribute name="NAME" x="34.29" y="-17.018" size="1.778" layer="95"/>
+</instance>
+<instance part="X_10" gate="G$1" x="53.34" y="-27.94" smashed="yes"/>
+<instance part="P+6" gate="VCC" x="53.34" y="-15.24" smashed="yes">
+<attribute name="VALUE" x="51.816" y="-14.224" size="1.27" layer="96"/>
 </instance>
 </instances>
@@
 <segment>
 <pinref part="DAC" gate="A" pin="LDAC"/>
-<wire x1="53.34" y1="5.08" x2="45.72" y2="5.08" width="0.127" layer="91"/>
-<wire x1="45.72" y1="5.08" x2="45.72" y2="2.54" width="0.127" layer="91"/>
+<wire x1="53.34" y1="5.08" x2="50.8" y2="5.08" width="0.127" layer="91"/>
+<wire x1="50.8" y1="5.08" x2="50.8" y2="2.54" width="0.127" layer="91"/>
 <pinref part="X_2" gate="G$1" pin="0"/>
 </segment>
@@
 <wire x1="-33.02" y1="45.72" x2="-35.56" y2="45.72" width="0.127" layer="91"/>
 <wire x1="-35.56" y1="45.72" x2="-35.56" y2="43.18" width="0.127" layer="91"/>
+</segment>
+<segment>
+<pinref part="ISP" gate="1" pin="1"/>
+<wire x1="45.72" y1="-25.4" x2="53.34" y2="-25.4" width="0.1524" layer="91"/>
+<wire x1="53.34" y1="-25.4" x2="53.34" y2="-27.94" width="0.1524" layer="91"/>
+<pinref part="X_10" gate="G$1" pin="0"/>
 </segment>
 </net>
@@
 <segment>
 <pinref part="DAC" gate="A" pin="VREF"/>
-<wire x1="83.82" y1="17.78" x2="88.9" y2="17.78" width="0.127" layer="91"/>
+<wire x1="83.82" y1="17.78" x2="86.36" y2="17.78" width="0.127" layer="91"/>
 <pinref part="P+1" gate="VCC" pin="VCC"/>
-<wire x1="88.9" y1="17.78" x2="88.9" y2="20.32" width="0.127" layer="91"/>
+<wire x1="86.36" y1="17.78" x2="86.36" y2="20.32" width="0.127" layer="91"/>
 </segment>
 <segment>
@@
 <wire x1="-33.02" y1="30.48" x2="-33.02" y2="35.56" width="0.127" layer="91"/>
 </segment>
+<segment>
+<pinref part="ISP" gate="1" pin="5"/>
+<wire x1="45.72" y1="-20.32" x2="53.34" y2="-20.32" width="0.1524" layer="91"/>
+<wire x1="53.34" y1="-20.32" x2="53.34" y2="-17.78" width="0.1524" layer="91"/>
+<pinref part="P+6" gate="VCC" pin="VCC"/>
+</segment>
 </net>
 <net name="N$2" class="0">
@@
 <wire x1="35.56" y1="15.24" x2="35.56" y2="63.5" width="0.127" layer="91"/>
 <wire x1="35.56" y1="63.5" x2="53.34" y2="63.5" width="0.127" layer="91"/>
+<wire x1="35.56" y1="15.24" x2="35.56" y2="-12.7" width="0.1524" layer="91"/>
+<wire x1="35.56" y1="-12.7" x2="27.94" y2="-12.7" width="0.1524" layer="91"/>
+<wire x1="27.94" y1="-12.7" x2="27.94" y2="-20.32" width="0.1524" layer="91"/>
+<pinref part="ISP" gate="1" pin="6"/>
+<wire x1="27.94" y1="-20.32" x2="30.48" y2="-20.32" width="0.1524" layer="91"/>
+<junction x="35.56" y="15.24"/>
 </segment>
 </net>
@@
 <wire x1="38.1" y1="10.16" x2="38.1" y2="12.7" width="0.127" layer="91"/>
 <junction x="38.1" y="12.7"/>
+<wire x1="38.1" y1="10.16" x2="38.1" y2="-12.7" width="0.1524" layer="91"/>
+<wire x1="38.1" y1="-12.7" x2="48.26" y2="-12.7" width="0.1524" layer="91"/>
+<wire x1="48.26" y1="-12.7" x2="48.26" y2="-22.86" width="0.1524" layer="91"/>
+<pinref part="ISP" gate="1" pin="3"/>
+<wire x1="48.26" y1="-22.86" x2="45.72" y2="-22.86" width="0.1524" layer="91"/>
+<junction x="38.1" y="10.16"/>
 </segment>
 </net>
@@
 <wire x1="40.64" y1="15.24" x2="40.64" y2="17.78" width="0.127" layer="91"/>
 <junction x="40.64" y="17.78"/>
+<wire x1="40.64" y1="15.24" x2="40.64" y2="-10.16" width="0.1524" layer="91"/>
+<wire x1="40.64" y1="-10.16" x2="25.4" y2="-10.16" width="0.1524" layer="91"/>
+<wire x1="25.4" y1="-10.16" x2="25.4" y2="-22.86" width="0.1524" layer="91"/>
+<pinref part="ISP" gate="1" pin="4"/>
+<wire x1="25.4" y1="-22.86" x2="30.48" y2="-22.86" width="0.1524" layer="91"/>
+<junction x="40.64" y="15.24"/>
 </segment>
 </net>
@@
 </segment>
 </net>
+<net name="N$22" class="0">
+<segment>
+<pinref part="ATMEGA48A" gate="IC" pin="PC6(!RESET!/PCINT14)"/>
+<wire x1="33.02" y1="43.18" x2="43.18" y2="43.18" width="0.1524" layer="91"/>
+<wire x1="43.18" y1="43.18" x2="43.18" y2="-7.62" width="0.1524" layer="91"/>
+<wire x1="43.18" y1="-7.62" x2="20.32" y2="-7.62" width="0.1524" layer="91"/>
+<wire x1="20.32" y1="-7.62" x2="20.32" y2="-25.4" width="0.1524" layer="91"/>
+<pinref part="ISP" gate="1" pin="2"/>
+<wire x1="20.32" y1="-25.4" x2="30.48" y2="-25.4" width="0.1524" layer="91"/>
+</segment>
+</net>
